File: eagle/RoomIndicator.Inside.Multiple.brd (EAGLE design)
At the start: 54 x 50 mm, 31 parts, among them IC1 MEGA328P, Q1 8MHz, T1 BC847, T2 BC847, T3 BC847, U1 3.3V/150mA

Commit message: Boards for printing
Parts:
- removed GREEN, RED: GREEN, led:LED5MM
- removed POWER: (no value), SparkFun-Connectors:1X02
- removed S1: (no value), SparkFun-Retired:TACTILE-PTH
- removed U1: 3.3V/150mA, SparkFun-PowerIC:SOT23-5
- added C10, C11, C12: 100n, rcl:C0805K
- added C13, C14: 27p, rcl:C0805K
- added D2: 1N4148, diode:DO35-7
- added IC2: MEGA328P, atmel:TQFP32-08
- added JP3, JP6: BATT, pinhead:1X02
- added JP4: NRF24L01, pinhead:2X04
- added JP5: SPI, SparkFun-Connectors:2X3
- added L2: 10uH, rcl:0204/7
- added LED1, LED2: GREEN, led:LED5MM
- added Q2: 8MHz, crystal:HC49/S
- added R10, R7: 10k, rcl:R0805
- added R8: 30, rcl:0204/5
- added R9: 5k-1M, rcl:0204/5
- added SP2: AL60PWIDE, buzzer:AL80P
- added T4: BC847, transistor:SOT23
- added U$2: (no value), holes:3,6
- C8: device rcl:C0805K -> rcl:C025-025X050
- C9: value 180p -> 100uF; device rcl:C0805K -> rcl:E2,5-5
- R5: value 30 -> 5k-1M
- moved C9 64.3 mm to (50.2, 68.0), flipped to the top
- moved R4 49.7 mm to (8.26, 77.5)
- moved T3 45.4 mm to (41.9, 80.0)
- moved C8 25.6 mm to (50.2, 63.5), flipped to the top, turned to 0 degrees
- moved R5 11.2 mm to (40.6, 31.1), turned to 180 degrees
- moved T1 4.07 mm to (41.9, 26.0)
- moved R3 3.18 mm to (46.4, 21.6)
- moved R2 2.93 mm to (40.6, 35.6), turned to 0 degrees
Connections:
- net BLUE renamed LED
- removed net N$1: POWER.2, U1.1, U1.3
- removed net N$2: R4.1, T3.1
- removed net N$3: RED.K, T3.3
- removed net N$7: R5.2, RED.A
- removed net N$8: C9.1, U1.4
- removed net RED: IC1.30, R4.2
- new net +3V1: C10.2, C8.1, C9.+, D2.C, IC2.4, IC2.6, JP4.1, JP5.2, JP6.1, L2.1, R4.2, R8.1, SP2.1
- new net AVCC1: C12.1, IC2.18, L2.2
- new net BUZZ1: IC2.2, R10.1
- new net CE1: IC2.25, JP4.4
- new net CSN1: IC2.14, JP4.3
- new net GND1: C10.1, C11.1, C12.2, C13.1, C14.1, C8.2, C9.-, IC2.21, IC2.3, IC2.5, JP4.2, JP5.6, JP6.2, R9.1, T3.2, T4.2
- new net INT2: IC2.1, R9.2
- new net INT3: IC2.32, JP4.7
- new net LED1: IC2.31, R7.2
- new net MISO1: IC2.16, JP4.8, JP5.1
- new net MOSI1: IC2.15, JP4.5, JP5.4
- new net N$14: C11.2, IC2.20
- new net N$15: R7.1, T3.1
- new net N$17: LED2.K, T3.3
- new net N$18: D2.A, SP2.2, T4.3
- new net N$19: R10.2, T4.1
- new net N$20: LED2.A, R8.2
- new net RST1: IC2.29, JP5.5, R4.1
- new net SCK1: IC2.17, JP4.6, JP5.3
- new net TOSC3: C14.2, IC2.8, Q2.1
- new net TOSC4: C13.2, IC2.7, Q2.2
- net +3V3: now also JP3.1; no longer R5.1, U1.5
- net GND: now also JP3.2, R5.1; no longer C8.1, C9.2, POWER.1, S1.3, S1.4, T3.2, U1.2
- net INT1: now also R5.2; no longer C8.2, S1.1, S1.2
- net N$11: now also LED1.K; no longer GREEN.K
- net N$6: now also LED1.A; no longer GREEN.A
Routing:
- net GND1: track 0.00 -> 212.3 mm, vias 0 -> 2
- net +3V1: track 0.00 -> 179.8 mm, vias 0 -> 5
- net GND: track 299.6 -> 212.3 mm
- net MOSI1: track 0.00 -> 66.5 mm, vias 0 -> 4
- net RST1: track 0.00 -> 57.2 mm, vias 0 -> 1
- net SCK1: track 0.00 -> 53.7 mm, vias 0 -> 2
- net MISO1: track 0.00 -> 49.6 mm, vias 0 -> 2
- net INT3: track 0.00 -> 45.7 mm, vias 0 -> 3
- net CSN1: track 0.00 -> 31.9 mm, vias 0 -> 3
- net CE1: track 0.00 -> 30.1 mm, vias 0 -> 1
- net AVCC1: track 0.00 -> 20.3 mm
- net INT1: track 25.9 -> 6.66 mm, vias 1 -> 0
- net TOSC3: track 0.00 -> 15.4 mm
- net N$19: track 4.00 -> 18.9 mm, vias 0 -> 2
- net TOSC4: track 0.00 -> 12.9 mm
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Other:
- board size 54 x 50 mm -> 54 x 104 mm
