File: eagle/RoomIndicator.Inside.brd (EAGLE design)
At the start: 54 x 50 mm, 24 parts, among them IC1 MEGA328P, Q1 8MHz, T1 BC847, T2 BC847

Commit message: Boards for printing
Parts:
- SP1: value AL60P -> AL60PWIDE; device buzzer:AL60P -> buzzer:AL80P
Routing:
- net N$16: track 16.9 -> 15.2 mm
- net +3V3: track 178.3 -> 179.8 mm
